File: MYC_devices_hardware/MYC_device_DTMF_Receiver/dtmf_rx.sch (EAGLE design)
At the start: 30 parts, among them IC1 MEGA8-P, IC2 7805T, Q1 20MHz, X1 8-15V, X2 1503_09, X3 1503_09

Commit message: some changes of DTMF devices
Parts:
- removed DC1: AM1S1203SZ, dc-dc-converter:NME
- removed L1, L2: 100u, inductor-neosid:MS85
- removed ST1: Power, pinhead:PINHD-1X6
- removed ST2: I2C, pinhead:PINHD-1X6
- removed ST3: SPI, pinhead:PINHD-1X8
- removed ST4: UART, pinhead:PINHD-1X8
- added C10, C9: 22u 1210, rcl:C-EUC1206
- added C11, C12: 100n, rcl:C-EU050-025X075
- added IC3: 7805TV, linear:7805TV
- added IC4: CM8870CP, california-micro-devices:CM8870CP
- added JP7, JP8: DTE/DCE, jumper:JP2E
- added JP9: USB, jumper:JP4E
- added LED1, LED2, LED3: PL006-WCY01, led:PL006-WCY01
- added Q2: 20MHz, special:XTAL/S
- added R1, R2, R8, R9: 4k7, resistor:R-EU_0207/5V
- added R5: 102k, resistor:R-EU_0207/5V
- added R6: 71,5k, resistor:R-EU_0207/5V
- added R7: 390k, resistor:R-EU_0207/5V
- added SL4: DTMF/RC5, con-amp-quick:M05
- added X4: RS232, con-subd:F09H
- C7, C8: value 22uF 1210 -> 22u 1210
- IC2: value 7805T -> MAX232; device linear:7805T -> maxim:MAX232
- JP2: value GND -> I2C
- JP3: value USB -> 5V; device jumper:JP4E -> jumper:JP1E
- JP5: value ISP -> Rs232-TTL; device jumper:JP3Q -> jumper:JP1E
- JP6: value USB2 -> ISP; device jumper:JP1E -> jumper:JP3Q
- R3: device resistor:R-EU_R1206 -> resistor:R-EU_0207/5V
- R4: value 4k7 -> -; device resistor:R-EU_R1206 -> resistor:R-EU_0207/5V
Connections:
- removed net VSS: C7.1, DC1.+VOUT, JP6.2, ST1.2
- new net C13: C7.1, IC2G$1.C1+
- new net N$11: IC2G$1.R2IN, JP7.1, JP8.3
- new net N$12: IC1.PD1(TXD), IC2G$1.T1IN, JP5.2, JP9.2
- new net N$13: C8.1, IC2G$1.C2+
- new net N$14: C7.2, IC2G$1.C1-
- new net N$16: C9.1, IC2G$1.V+
- new net N$17: C10.2, IC2G$1.V-
- new net N$21: C11.1, SL4.1
- new net N$23: IC1.PD4(XCK/T0), R2.2
- new net N$24: C11.2, R5.1
- new net N$25: IC4.IN-, R4.2, R5.2, R6.2
- new net N$26: IC4.GS, R4.1, R6.1
- new net N$29: IC4.OSC2, Q2.1
- new net N$30: IC1.PC1(ADC1), IC4.Q3
- new net N$31: IC4.OSC1, Q2.2
- new net N$32: IC4.EST, R7.2
- new net N$34: IC1.PC3(ADC3), IC4.Q1
- new net N$38: IC1.PC2(ADC2), IC4.Q2
- new net N$40: C12.2, IC4.ST/GT, R7.1
- new net N$42: IC1.PD2(INT0), IC4.STD
- new net N$48: LED3.C, R3.1
- new net N$49: LED2.C, R2.1
- new net N$50: LED1.C, R1.1
- new net N$51: IC1.PD3(INT1), R3.2
- net GND: now also C10.1, IC2G$1.R1IN, IC2G$1.T2IN, IC2P.GND, IC3.GND, IC4.INH, IC4.VSS, IC4.VSS@1, JP3.2, JP6.6, JP9.3, SL4.5, X4.5; no longer C7.2, C8.2, DC1.-VIN, DC1.-VOUT, IC2.GND, JP2.1, JP2.2, JP3.4, JP5.6, ST1.4, ST1.5, ST3.2
- net N$1: now also IC1.PD6(AIN0), R1.2; no longer IC1.PC0(ADC0), ST4.5
- net N$10: now also IC2G$1.T1OUT, JP7.3, JP8.1; no longer IC1.PB1(OC1A), ST2.6
- net N$15: now also JP6.1; no longer JP5.1, ST3.4
- net N$18: now also JP6.5; no longer JP5.5
- net N$2: now also IC1.PD0(RXD), IC2G$1.R2OUT, JP5.1, JP9.1; no longer IC1.PB0(ICP), ST2.5
- net N$20: now also JP6.3; no longer JP5.3, ST3.3
- net N$22: now also JP2.2, R9.2; no longer R4.2
- net N$28: now also JP6.4; no longer JP5.4, ST3.5
- net N$3: now also C8.2, IC2G$1.C2-; no longer C8.1, DC1.+VIN, L1.2
- net N$33: now also D1.C, IC3.VI; no longer IC2.VI, L2.2
- net N$4: now also JP8.2, X4.2; no longer IC1.PB2(SS/OC1B), ST3.6
- net N$44: now also JP6.2; no longer JP5.2
- net N$5: now also JP2.1, R8.2; no longer R3.2
- net N$6: now also IC1.PB0(ICP); no longer IC1.PD7(AIN1)
- net N$7: now also IC4.IN+, IC4.VREF; no longer D1.C, L1.1, L2.1
- net N$8: now also IC1.PC0(ADC0), IC4.Q4; no longer IC1.PD1(TXD), JP3.3
- net N$9: now also JP7.2, X4.3; no longer IC1.PD0(RXD), JP3.2
- net VDD: now also C12.1, C9.2, IC2P.VCC, IC3.VO, IC4.TOE, IC4.VDD, JP3.1, JP9.4, LED1.A, LED2.A, LED3.A, R8.1, R9.1; no longer IC2.VO, JP6.1, R3.1, R4.1, ST1.3
Other:
- moved on the sheet: C1, C2, C7, C8, D1, JP2, JP4, R3, R4, X1
