File: MYC_devices_hardware/MYC_eletronic_load/electronic_load.sch (EAGLE design)
At the start: 58 parts, among them IC1 MEGA8-P, IC2 MAX232, IC3 7805TV, Q1 20MHz, T1 BC817 SOT23, T2 BC817 SOT23, T3 BC817 SOT23, T4 BC807 SOT23, T5 BC817 SOT23, T6 BC817 SOT23, X1 8-15V, X2 1503_09, X3 1503_09, X4 RS232

Commit message: Electronic load added; error correction and minor enhancements for I2C Interface
Parts:
- removed JP8: DTE/DCE, jumper:JP2E
- removed JP9: USB, jumper:JP4E
- removed LED2, LED3, LED4: PL006-WCY01, led:PL006-WCY01
- removed SL3: GPO, con-amp-quick:M05
- removed T3, T5, T6: BC817 SOT23, transistor:BC817-NPN-SOT23-BEC
- removed T4: BC807 SOT23, transistor-pnp:BC807-25SMD
- added C13, C14, C15, C16, C17, C18, C19, C20, C21, C22, C23, C24, C25, C26, C27: 22uF 1210, rcl:C-EUC1206
- added C28: 1u, resistor:C-EUC1206
- added IC10, IC4, IC5, IC6, IC7, IC8, IC9: MCP4921, dac:MCP491
- added IC11, IC12: LM324N, linear:LM324N
- added IC13: 78L5, v-reg:78LXX
- added IC14, IC15, IC16, IC17, IC18, IC19, IC20: MCP603CH, linear:MCP603CH
- added JP5: Rs232-TTL, jumper:JP1E
- added L1: 22u, inductor-neosid:MS85
- added R14: 12k, resistor:R-EU_R1206
- added R17, R34: 8k2, resistor:R-EU_R1206
- added R18, R20, R22, R24, R26, R30, R32, R38, R40, R42, R44, R47, R48, R50: 154k, resistor:R-EU_0207/2V
- added R19, R21, R23, R25, R27, R31, R33, R39, R41, R43, R45, R46, R49, R51: 18k, resistor:R-EU_0207/2V
- added R28: 1k5, resistor:R-EU_R1206
- added R29: 180, resistor:R-EU_R1206
- added R35: 18k, resistor:R-EU_R1206
- added R36, R37: 10k, resistor:R-EU_R1206
- added SL5: Iin, con-amp-quick:M05
- added SL6: U/Iin, con-amp-quick:M05
- C10, C9: value 22u 1210 -> 22uF 1210
- C11: value 10n -> 22uF 1210; device resistor:C-EU050-025X075 -> rcl:C-EUC1206
- C12: value 10nF -> 22uF 1210; device resistor:C-EU050-025X075 -> rcl:C-EUC1206
- C2, C3: value 22uF 1210 -> 18pF; device rcl:C-EUC1206 -> resistor:C-EU025-025X050
- C4: value 18pF -> 22uF 1210; device resistor:C-EU025-025X050 -> rcl:C-EUC1206
- C5: value 18pF -> 22u 1210; device resistor:C-EU025-025X050 -> rcl:C-EUC1206
- C6: value 22uF 1210 -> 22u 1210
- IC1: value MEGA8-P -> MEGA16-P; device atmel:MEGA8-P -> atmel:MEGA16-P
- IC3: value 7805TV -> 79L09; device linear:7805TV -> v-reg:78LXX
- JP7: value DTE/DCE -> USB; device jumper:JP2E -> jumper:JP4E
- R1, R2: device resistor:R-EU_R1206 -> resistor:R-EU_0207/2V
- R10, R12, R4: value 4k7 -> 12k
- R11, R15: value 4k7 -> 8k2
- R13: value 10k -> 8k2
- R16: value 10k -> 12k
- R5, R7: value 10k -> 8k2; device resistor:R-EU_0207/2V -> resistor:R-EU_R1206
- R6: value 10 -> 12k; device resistor:R-EU_0207/2V -> resistor:R-EU_R1206
- R8: value 4k7 -> 12k; device resistor:R-EU_0207/2V -> resistor:R-EU_R1206
- R9: value 4k7 -> 8k2; device resistor:R-EU_0207/2V -> resistor:R-EU_R1206
- SL1: value GPIO1 -> Gates1
- SL2: value GPIO2 -> Gates2
- SL4: value DTMF/RC5 -> Iin
- T1: value BC817 SOT23 -> BC807; device transistor:BC817-NPN-SOT23-BEC -> transistor:BC807-16-PNP-SOT23-BEC
- T2: value BC817 SOT23 -> BC817; device transistor:BC817-NPN-SOT23-BEC -> transistor:BC817-16-NPN-SOT23-BEC
Connections:
- new net 9V: C27.1, IC13.IN, IC3.OUT, R34.1
- new net FET1: IC12C.OUT, R16.2, SL2.3
- new net FET2: IC12A.OUT, R12.2, SL2.2
- new net FET3: IC12D.OUT, R14.2, SL2.1
- new net FET4: IC11B.OUT, R6.2, SL1.4
- new net FET5: IC11C.OUT, R8.2, SL1.3
- new net FET6: IC11A.OUT, R4.2, SL1.2
- new net FET7: IC11D.OUT, R10.2, SL1.1
- new net GON: IC1.(OC1A)PD5, R36.1
- new net I1: IC1.(ADC1)PA1, IC14.OUT, R18.2
- new net I2: IC1.(ADC2)PA2, IC15.OUT, R20.2
- new net I3: IC1.(ADC3)PA3, IC16.OUT, R22.2
- new net I4: IC1.(ADC4)PA4, IC17.OUT, R24.2
- new net I5: IC1.(ADC5)PA5, IC18.OUT, R26.2
- new net I6: IC1.(ADC6)PA6, IC19.OUT, R30.2
- new net I7: IC1.(ADC7)PA7, IC20.OUT, R32.2
- new net N$36: IC11D.-IN, R10.1, R11.1
- new net N$40: IC12D.-IN, R14.1, R15.1
- new net N$54: R25.2, SL5.3
- new net N$55: IC5A.VOUT, R7.2
- new net N$56: C26.1, D1.C, IC3.IN, T1.E
- new net N$57: IC12A.-IN, R12.1, R13.1
- new net N$58: IC12C.-IN, R16.1, R17.1
- new net N$59: C24.1, C25.1, IC11P.V+, IC12P.V+, T1.C
- new net N$60: R27.2, SL5.5
- new net N$61: R37.2, T1.B
- new net N$62: IC1.(TOSC1)PC6, IC5A.CS
- new net N$63: R37.1, T2.C
- new net N$64: R36.2, T2.B
- new net N$65: R38.1, SL4.1
- new net N$66: R40.1, SL4.3
- new net N$67: IC14.+IN, R38.2, R39.1
- new net N$68: R42.2, SL4.5
- new net N$69: R19.2, SL4.2
- new net N$70: R44.1, SL5.2
- new net N$71: IC1.(TDI)PC5, IC6A.CS
- new net N$72: IC18.+IN, R46.1, R47.2
- new net N$73: IC11B.-IN, R6.1, R7.1
- new net N$74: IC19.+IN, R48.2, R49.1
- new net N$76: R50.1, SL6.3
- new net N$79: R23.2, SL5.1
- new net N$80: IC16.+IN, R42.1, R43.1
- new net N$89: R33.2, SL6.4
- new net N$90: IC20.+IN, R50.2, R51.1
- new net N$91: IC11A.-IN, R4.1, R5.1
- new net N$96: IC12B.-IN, IC12B.OUT
- new net U: C28.1, IC1.(ADC0)PA0, R28.1, R29.1
- new net VREF: IC11A.+IN, IC11B.+IN, IC11C.+IN, IC11D.+IN, IC12A.+IN, IC12C.+IN, IC12D.+IN, R34.2, R35.1
- net C13: now also C5.1; no longer C7.1
- net GND: now also C1.1, C10.2, C11.2, C13.2, C14.2, C15.2, C16.2, C17.2, C18.2, C19.2, C2.1, C20.2, C21.2, C22.2, C23.2, C24.2, C25.2, C26.2, C27.2, C28.2, C4.2, C8.1, C9.2, IC10P.GND, IC11P.V-, IC12B.+IN, IC12P.V-, IC13.GND, IC14.!CS, IC14.V-, IC15.!CS, IC15.V-, IC16.!CS, IC16.V-, IC17.!CS, IC17.V-, IC18.!CS, IC18.V-, IC19.!CS, IC19.V-, IC20.!CS, IC20.V-, IC2G$1.R2IN, IC4P.GND, IC5P.GND, IC6P.GND, IC7P.GND, IC8P.GND, IC9P.GND, JP7.3, R28.2, R35.2, R39.2, R41.2, R43.2, R45.2, R46.2, R49.2, R51.2, SL2.4; no longer C1.2, C10.1, C2.2, C4.1, C5.1, C6.2, IC2G$1.R1IN, JP9.3, SL3.5, SL4.5, T1.E, T3.E, T5.E, T6.E
- net N$1: now also IC14.-IN, R18.1, R19.1; no longer IC1.PD7(AIN1), R1.2
- net N$10: now also IC6A.VOUT, R9.2; no longer IC2G$1.T1OUT, JP7.3, JP8.1
- net N$11: now also IC1.(ICP)PD6, IC10A.LDAC, IC4A.LDAC, IC5A.LDAC, IC6A.LDAC, IC7A.LDAC, IC8A.LDAC, IC9A.LDAC; no longer IC1.PC0(ADC0), SL1.1, T6.C
- net N$12: now also D1.A, L1.2; no longer IC1.PD1(TXD), IC2G$1.T1IN, JP9.2
- net N$13: now also C6.1; no longer C8.1
- net N$14: now also C5.2; no longer C7.2
- net N$15: now also IC1.(MISO)PB6; no longer IC1.PB4(MISO)
- net N$16: now also C7.1; no longer C9.1
- net N$17: now also C8.2; no longer C10.2
- net N$18: now also IC1.RESET; no longer IC1.PC6(/RESET)
- net N$19: now also C2.2, IC1.XTAL2; no longer C4.2, IC1.PB6(XTAL1/TOSC1)
- net N$2: now also IC1.(RXD)PD0, IC2G$1.R1OUT, JP5.1, JP7.1; no longer IC1.PD0(RXD), IC2G$1.R2OUT, JP9.1
- net N$20: now also IC1.(MOSI)PB5, IC10A.SDI, IC4A.SDI, IC5A.SDI, IC6A.SDI, IC7A.SDI, IC8A.SDI, IC9A.SDI, JP6.4; no longer IC1.PB5(SCK), JP6.3
- net N$21: now also IC7A.VOUT, R11.2; no longer IC1.PD5(T1), SL2.1
- net N$22: now also IC1.(SCL)PC0, R2.2; no longer IC1.PC5(ADC5/SCL), R9.2
- net N$23: now also IC1.(TMS)PC3, IC8A.CS; no longer IC1.PD4(XCK/T0), R10.2, R2.2, SL2.2
- net N$24: now also IC8A.VOUT, R13.2; no longer R12.1, T3.B
- net N$25: now also C4.1, IC1.AVCC, IC1.VCC, JP1.1, JP6.2; no longer IC1.PC1(ADC1), R16.1, SL1.2
- net N$26: now also IC9A.VOUT, R15.2; no longer IC1.PC2(ADC2), SL1.3
- net N$27: now also R29.2, SL6.5; no longer D1.A, X1.-1
- net N$28: now also IC1.(SCK)PB7, IC10A.SCK, IC4A.SCK, IC5A.SCK, IC6A.SCK, IC7A.SCK, IC8A.SCK, IC9A.SCK, JP6.3; no longer IC1.PB3(MOSI/OC2), JP6.4
- net N$29: now also R21.2, SL4.4; no longer C11.2, R5.1, T4.B
- net N$3: now also C6.2; no longer C8.2
- net N$30: now also IC15.-IN, R20.1, R21.1; no longer C11.1, IC1.PB1(OC1A), R5.2, R7.1
- net N$31: now also IC4A.VOUT, R5.2; no longer R6.2, T4.C
- net N$32: now also IC20.-IN, R32.1, R33.1; no longer C12.1, R6.1, R7.2, SL4.1
- net N$33: now also IC2G$1.T1OUT, X4.2; no longer C1.1, D1.C, IC3.VI
- net N$34: now also IC19.-IN, R30.1, R31.1; no longer R11.1, T2.B
- net N$35: now also C1.2; no longer C3.2
- net N$37: now also C3.2, IC1.XTAL1; no longer C5.2, IC1.PB7(XTAL2/TOSC2)
- net N$38: now also IC11C.-IN, R8.1, R9.1; no longer R16.2, T5.B
- net N$39: now also IC10A.VOUT, R17.2; no longer IC1.PC3(ADC3), SL1.4
- net N$4: now also IC1.(OC2)PD7, IC10A.CS; no longer JP8.2, X4.2
- net N$41: now also IC16.-IN, R22.1, R23.1; no longer IC2G$1.R2IN, JP7.1, JP8.3
- net N$42: now also IC1.(T0/XCK)PB0, R3.1; no longer R13.1, T6.B
- net N$43: now also LED1.C, R3.2; no longer LED4.C, R4.1
- net N$44: now also IC17.+IN, R44.2, R45.1; no longer C6.1, IC1.AVCC, IC1.VCC@1, JP1.1, JP6.2
- net N$45: now also IC17.-IN, R24.1, R25.1; no longer SL3.2, T1.C
- net N$46: now also IC1.(T1)PB1, JP4.1; no longer SL3.3, T2.C
- net N$47: now also IC18.-IN, R26.1, R27.1; no longer SL3.4, T3.C
- net N$48: now also R47.1, SL5.4; no longer LED3.C, R3.1
- net N$49: now also IC15.+IN, R40.2, R41.1; no longer LED2.C, R2.1
- net N$5: now also IC1.(SDA)PC1, R1.2; no longer IC1.PC4(ADC4/SDA), R8.2
- net N$50: now also IC1.(TOSC2)PC7, IC4A.CS; no longer LED1.C, R1.1
- net N$51: now also IC1.(TDO)PC4, IC7A.CS; no longer IC1.PD3(INT1), R11.2, R3.2, SL2.3
- net N$52: now also R48.1, SL6.1; no longer IC1.PD2(INT0), R12.2, R4.2, SL2.4
- net N$53: now also R31.2, SL6.2; no longer R13.2, R15.2, SL4.3, T5.C
- net N$6: now also IC1.(TXD)PD1, IC2G$1.T1IN, JP5.2, JP7.2; no longer IC1.PB2(SS/OC1B), JP4.1
- net N$7: now also L1.1, X1.-1; no longer IC1.PB0(ICP), SL4.2
- net N$8: now also IC1.(TCK)PC2, IC9A.CS; no longer R10.1, T1.B
- net N$9: now also IC2G$1.R1IN; no longer JP7.2
- net VDD: now also C10.1, C11.1, C12.1, C13.1, C14.1, C15.1, C16.1, C17.1, C18.1, C19.1, C20.1, C21.1, C22.1, C23.1, C7.2, C9.1, IC10A.VREF, IC10P.VCC, IC13.OUT, IC14.V+, IC15.V+, IC16.V+, IC17.V+, IC18.V+, IC19.V+, IC20.V+, IC4A.VREF, IC4P.VCC, IC5A.VREF, IC5P.VCC, IC6A.VREF, IC6P.VCC, IC7A.VREF, IC7P.VCC, IC8A.VREF, IC8P.VCC, IC9A.VREF, IC9P.VCC, JP7.4, R1.1, R2.1; no longer C2.1, C9.2, IC3.VO, JP9.4, LED2.A, LED3.A, LED4.A, R15.1, R8.1, R9.1, SL3.1, SL4.4, T4.E
Other:
- note added: "+ extern 51k for 90V"
