File: MYC_devices_hardware/MYC_device_Textdisplay/textdisplay.brd (EAGLE design)
At the start: 61 x 39.4 mm, 26 parts, among them IC1 MEGA8-P, IC2 7805T, Q1 20MHz, Q2 BC307, X1 8-15V, X2 1503_09, X3 1503_09

Commit message: board slightly modifie, minor firmware updates
Parts:
- removed JP5: GND, jumper:JP1
- IC2: value 7805T -> 78L05; device linear:TO220H -> v-reg:78LXX
- moved JP3 23.5 mm to (75.6, 8.89), turned to 90 degrees
- moved IC2 8.98 mm to (26.0, 22.2), turned to 180 degrees
- moved R1 1.27 mm to (57.8, 23.5), turned to 180 degrees
- moved JP2 1.27 mm to (76.2, 27.9)
- moved R2 1.27 mm to (51.4, 23.5)
- moved SL1 0.64 mm to (50.2, 4.45)
- moved SL2 0.64 mm to (29.8, 4.45)
- turned C7 to 0 degrees
Connections:
- net GND: now also IC2.GND; no longer IC2.2, JP5.1, JP5.2
- net N$18: now also IC2.IN; no longer IC2.1
- net VDD: now also IC2.OUT; no longer IC2.3
Routing:
- net E: track 120.7 -> 65.1 mm
- net VDD: track 95.7 -> 116.0 mm, vias 1 -> 0
- net MOSI: track 15.7 -> 29.5 mm, vias 1 -> 0
- net D5: track 66.6 -> 55.0 mm, vias 3 -> 0
- net D6: track 108.7 -> 98.5 mm
- net D7: track 75.5 -> 66.2 mm, vias 5 -> 2
- net N$4: track 50.5 -> 58.3 mm, vias 1 -> 0
- net RESET: track 52.5 -> 58.4 mm, vias 1 -> 0
- net TXD: track 21.0 -> 25.9 mm
- net SCL: track 35.2 -> 40.0 mm
- net CONTRAST: track 52.4 -> 48.1 mm
- net SDA: track 37.7 -> 33.9 mm
- net MISO: track 16.0 -> 12.2 mm
- net GND: track 201.0 -> 197.7 mm
- net N$37: track 11.0 -> 14.0 mm
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- added copper zone on layer 1, net GND
- removed copper zone on layer 1, net VDD
Other:
- board text added: "V01.3"
- board text removed: "V01.1"
