File: MYC_devices_hardware/MYC_device_Textdisplay/textdisplay.sch (EAGLE design)
At the start: 26 parts, among them IC1 MEGA8-P, IC2 7805T, Q1 20MHz, Q2 BC307, X1 8-15V, X2 1503_09, X3 1503_09

Commit message: board slightly modifie, minor firmware updates
Parts:
- removed JP5: GND, jumper:JP1E
- IC2: value 7805T -> 78L05; device linear:7805T -> v-reg:78LXX
Connections:
- net GND: no longer JP5.1, JP5.2
- net N$18: now also IC2.IN; no longer IC2.VI
- net VDD: now also IC2.OUT; no longer IC2.VO
Changed lines of the file:
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@@
 </classes>
 <parts>
-<part name="IC2" library="linear" deviceset="78*" device="T" technology="05"/>
 <part name="C1" library="resistor" deviceset="C-EU" device="C1206" value="22u"/>
 <part name="C2" library="resistor" deviceset="C-EU" device="C1206" value="22u"/>
@@
 <part name="VDD6" library="supply1" deviceset="VDD" device=""/>
 <part name="X1" library="con-conrad" deviceset="737992-55" device="" value="8-15V"/>
-<part name="JP5" library="jumper" deviceset="JP1E" device="" value="GND"/>
 <part name="D1" library="diode" deviceset="1N4004" device=""/>
 <part name="JP3" library="jumper" deviceset="JP1E" device="" value="Reset"/>
@@
 <part name="R5" library="resistor" deviceset="R-EU_" device="0207/2V" value="4k7"/>
 <part name="VDD5" library="supply1" deviceset="VDD" device=""/>
+<part name="IC2" library="v-reg" deviceset="78LXX" device="" value="78L05"/>
 </parts>
 <sheets>
@@
 </plain>
 <instances>
-<instance part="IC2" gate="A1" x="99.06" y="83.82"/>
 <instance part="C1" gate="G$1" x="73.66" y="81.28"/>
 <instance part="C2" gate="G$1" x="121.92" y="81.28"/>
@@
 <instance part="VDD6" gate="G$1" x="162.56" y="317.5"/>
 <instance part="X1" gate="G$1" x="20.32" y="81.28" rot="R180"/>
-<instance part="JP5" gate="A" x="167.64" y="78.74"/>
 <instance part="D1" gate="1" x="35.56" y="83.82"/>
 <instance part="JP3" gate="A" x="132.08" y="213.36"/>
@@
 <instance part="R5" gate="G$1" x="167.64" y="233.68" rot="R90"/>
 <instance part="VDD5" gate="G$1" x="185.42" y="215.9"/>
+<instance part="IC2" gate="1" x="101.6" y="83.82"/>
 </instances>
 <busses>
@@
 <junction x="121.92" y="83.82"/>
 <junction x="121.92" y="83.82"/>
-<pinref part="IC2" gate="A1" pin="VO"/>
 <pinref part="C2" gate="G$1" pin="1"/>
 <wire x1="121.92" y1="83.82" x2="154.94" y2="83.82" width="0.1524" layer="91"/>
+<pinref part="IC2" gate="1" pin="OUT"/>
 </segment>
 <segment>
@@
 <net name="GND" class="0">
 <segment>
-<wire x1="73.66" y1="76.2" x2="99.06" y2="76.2" width="0.1524" layer="91"/>
-<wire x1="99.06" y1="76.2" x2="101.6" y2="76.2" width="0.1524" layer="91"/>
+<wire x1="73.66" y1="76.2" x2="101.6" y2="76.2" width="0.1524" layer="91"/>
 <wire x1="101.6" y1="76.2" x2="121.92" y2="76.2" width="0.1524" layer="91"/>
 <wire x1="101.6" y1="76.2" x2="101.6" y2="73.66" width="0.1524" layer="91"/>
-<wire x1="121.92" y1="76.2" x2="167.64" y2="76.2" width="0.1524" layer="91"/>
-<junction x="99.06" y="76.2"/>
 <junction x="101.6" y="76.2"/>
-<junction x="121.92" y="76.2"/>
 <pinref part="C1" gate="G$1" pin="2"/>
-<pinref part="IC2" gate="A1" pin="GND"/>
 <pinref part="C2" gate="G$1" pin="2"/>
 <pinref part="GND4" gate="1" pin="GND"/>
-<wire x1="167.64" y1="76.2" x2="170.18" y2="76.2" width="0.1524" layer="91"/>
-<junction x="167.64" y="76.2"/>
-<pinref part="JP5" gate="A" pin="1"/>
-<pinref part="JP5" gate="A" pin="2"/>
-<junction x="170.18" y="76.2"/>
 <pinref part="X1" gate="G$1" pin="+"/>
 <pinref part="X1" gate="G$1" pin="K"/>
@@
 <junction x="73.66" y="76.2"/>
 <junction x="25.4" y="78.74"/>
+<pinref part="IC2" gate="1" pin="GND"/>
 </segment>
 <segment>
@@
 <net name="N$18" class="0">
 <segment>
-<pinref part="IC2" gate="A1" pin="VI"/>
-<wire x1="73.66" y1="83.82" x2="88.9" y2="83.82" width="0.1524" layer="91"/>
+<wire x1="73.66" y1="83.82" x2="93.98" y2="83.82" width="0.1524" layer="91"/>
 <pinref part="C1" gate="G$1" pin="1"/>
 <pinref part="L1" gate="G$1" pin="2"/>
 <wire x1="60.96" y1="83.82" x2="73.66" y2="83.82" width="0.1524" layer="91"/>
 <junction x="73.66" y="83.82"/>
-</segment>
-</net>
+<pinref part="IC2" gate="1" pin="IN"/>
+</segment>
+</net>
