File: MYC_devices_hardware/MYCdevice_i2c_rs232_interface/i2c_rs232_interface.sch (EAGLE design)
At the start: 58 parts, among them IC1 MEGA8-P, IC2 MAX232, IC3 7805TV, Q1 20MHz, T1 BC817 SOT23, T2 BC817 SOT23, T3 BC817 SOT23, T4 BC807 SOT23, T5 BC817 SOT23, T6 BC817 SOT23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

Commit message: new connectors, I2c with 3V
Parts:
- removed T5, T6: BC817 SOT23, transistor:BC817-NPN-SOT23-BEC
- removed X3: 1503_09, con-lumberg:1503_09
- removed X4: RS232, con-subd:F09H
- added IC4: 78L05, v-reg:78LXX
- added JP5: Reset, jumper:JP1E
- added R14: 10k, resistor:R-EU_R1206
- added SL5: GPIO1, con-amp-quick:M05
- added SL6: GPIO2, con-amp-quick:M05
- C1, C2, C6: value 22uF 1210 -> 22u
- C10: value 22u 1210 -> 22uF
- C11, C12: device resistor:C-EU050-025X075 -> resistor:C-EUC1206
- C7, C8, C9: value 22u 1210 -> 22u
- IC1: value MEGA8-P -> MEGA8-AI; device atmel:MEGA8-P -> atmel:MEGA8-AI
- IC3: value 7805TV -> PCA9517; device linear:7805TV -> PCA9517:PCA9517
- JP11: value ISP -> (none)
- JP2: value I2C -> 3V/5V; device jumper:JP1E -> jumper:JP2E
- JP3: value 5V -> SDA
- JP4: value Reset -> SCL
- JP7: value DTE/DCE -> USB; device jumper:JP2E -> jumper:JP4E
- JP9: value USB -> DTE/DCE; device jumper:JP4E -> jumper:JP2E
- R1, R2, R3, R4: value 4k7 -> see manual
- R13: value 10k -> 4k7
- R15: value 4k7 -> 10k
- R16: value 10k -> 10
- R5: value 10k -> 1k; device resistor:R-EU_0207/2V -> resistor:R-EU_R1206
- R6: value 10 -> 1k5; device resistor:R-EU_0207/2V -> resistor:R-EU_R1206
- R7: value 10k -> 4k7; device resistor:R-EU_0207/2V -> resistor:R-EU_R1206
- R8, R9: device resistor:R-EU_0207/2V -> resistor:R-EU_R1206
- SL1: value GPIO1 -> I2C1; device con-amp-quick:M05 -> con-amp-quick:M03
- SL2: value GPIO2 -> I2C2; device con-amp-quick:M05 -> con-amp-quick:M03
- X2: value 1503_09 -> RS232; device con-lumberg:1503_09 -> con-subd:F09H
- renumbered JP6 to JP11
Connections:
- removed net N$42 (its old number): R13.1, T6.B
- new net N$36: IC1.PC1(ADC1), SL5.2
- new net N$40: IC1.PD3(INT1), SL6.3
- new net N$54: IC1.ADC7, SL6.2
- new net N$56: IC3.VCCA, JP2.2, R1.1, R2.1
- new net N$7: IC1.PC2(ADC2), SL5.1
- net C13: now also C6.1; no longer C7.1
- net GND: now also C10.2, C9.1, IC1.GND@2, IC4.GND, JP5.2, JP7.3, R6.2, SL1.1, SL2.1, SL5.5, SL6.5, X2.5; no longer C10.1, C6.2, JP3.2, JP4.2, JP9.3, SL1.5, SL2.5, T5.E, T6.E, X2.1, X3.1, X4.5
- net N$1: now also R7.2; no longer R1.2
- net N$10: now also JP8.3, JP9.1; no longer JP7.3, JP8.1
- net N$11: now also C10.1, IC1.AVCC, IC1.VCC@1, IC1.VCC@2, JP1.1, JP11.2; no longer IC1.PC0(ADC0), SL1.1, T6.C
- net N$12: now also JP7.2; no longer JP9.2
- net N$13: now also C7.1; no longer C8.1
- net N$14: now also C6.2; no longer C7.2
- net N$16: now also C8.1; no longer C9.1
- net N$17: now also C9.2; no longer C10.2
- net N$2: now also JP7.1; no longer JP9.1
- net N$21: now also IC1.ADC6, SL6.1; no longer IC1.PD5(T1), SL2.1
- net N$22: now also IC3.SCLB, JP4.2, R3.2; no longer JP2.2, R9.2, X2.2, X3.2
- net N$23: now also IC1.PD6(AIN0), R11.2, R8.2; no longer IC1.PD4(XCK/T0), R10.2, R2.2, SL2.2
- net N$24: now also R13.1; no longer R12.1
- net N$25: now also IC1.PD5(T1), R12.2, R9.2; no longer IC1.PC1(ADC1), R16.1, SL1.2
- net N$26: now also IC1.PC0(ADC0), SL5.3; no longer IC1.PC2(ADC2), SL1.3
- net N$29: now also R14.1; no longer R5.1
- net N$3: now also C7.2; no longer C8.2
- net N$30: now also R14.2, R15.1; no longer R5.2, R7.1
- net N$31: now also R16.2; no longer R6.2
- net N$32: now also R15.2, R16.1; no longer R6.1, R7.2
- net N$33: now also IC4.IN; no longer IC3.VI
- net N$34: now also R12.1; no longer R11.1
- net N$38: now also IC3.SCLA, JP4.1, R2.2, SL1.2, SL2.2; no longer R16.2, T5.B
- net N$39: now also SL5.4; no longer SL1.4
- net N$4: now also JP9.2, X2.2; no longer JP8.2, X4.2
- net N$41: now also JP8.1, JP9.3; no longer JP7.1, JP8.3
- net N$43: now also R10.1; no longer R4.1
- net N$44: now also IC3.SDAA, JP3.1, R1.2, SL1.3, SL2.3; no longer C6.1, IC1.AVCC, IC1.VCC@1, JP1.1, JP11.2
- net N$48: now also R9.1; no longer R3.1
- net N$49: now also R8.1; no longer R2.1
- net N$5: now also IC3.SDAB, JP3.2, R4.2; no longer JP2.1, R8.2, X2.3, X3.3
- net N$50: now also R7.1; no longer R1.1
- net N$51: now also IC1.PD2(INT0), SL6.4; no longer IC1.PD3(INT1), R11.2, R3.2, SL2.3
- net N$52: now also IC1.PD4(XCK/T0), R10.2, R13.2; no longer IC1.PD2(INT0), R12.2, R4.2, SL2.4
- net N$53: now also JP2.1, R5.2, R6.1; no longer R13.2, R15.2, SL4.3, T5.C
- net N$6: now also JP5.1; no longer JP4.1
- net N$8: now also R11.1; no longer R10.1
- net N$9: now also JP8.2, X2.3; no longer JP7.2, X4.3
- net VDD: now also C8.2, IC3.EN, IC3.VCCB, IC4.OUT, JP2.3, JP7.4, R3.1, R4.1, R5.1; no longer C9.2, IC3.VO, JP3.1, JP9.4, R15.1, R8.1, R9.1
Other:
- moved on the sheet: C1, C10, C2, C6, C7, C8, C9, D1, JP1, JP3, JP4, JP8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
