File: MYC_devices_hardware/MYCdevice_DTMF_Transceiver/dtmf_trx.sch (EAGLE design)
At the start: 33 parts, among them IC1 78L05Z, IC2 MT8880, IC4 MEGA8-P, Q1 20MHz, Q2 3,579545MHz, X1 8-15V, X2 1503_09, X3 1503_09

Commit message: new board
Parts:
- removed LED1: PL006-WCY01, led:PL006-WCY01
- removed SL1: DTMF, con-amp-quick:M05
- removed X2, X3: 1503_09, con-lumberg:1503_09
- added C11, C12: 100n, resistor:C-EU050-025X075
- added C13: 10n, resistor:C-EU050-025X075
- added IC3: PCA9517, PCA9517:PCA9517
- added IC5: MT8880, dk1ri:MT8880
- added JP4: SCL, jumper:JP1E
- added JP6: ISP, jumper:JP3Q
- added JP7: RS232-USB, jumper:JP4E
- added R11: 10k, resistor:R-EU_R1206
- added R5: 1k, resistor:R-EU_R1206
- added R6: 1k5, resistor:R-EU_R1206
- added SL2, SL3: I2c, con-amp-quick:M03
- added SL4: DTMF, con-amp-quick:M03
- added X4: RS232, con-subd:F09H
- C4: value 22uF -> 18pF; device rcl:C-EUC1206 -> resistor:C-EU025-025X050
- C6: value 18pF -> 22uF; device resistor:C-EU025-025X050 -> rcl:C-EUC1206
- C7, C8: value 100n -> 22uF; device resistor:C-EU050-025X075 -> rcl:C-EUC1206
- C9: value 10n -> 22uF; device resistor:C-EU050-025X075 -> rcl:C-EUC1206
- IC1: value 78L05Z -> MEGA328; device linear:78L05Z -> atmel:MEGA8-P
- IC2: value MT8880 -> MAX232; device dk1ri:MT8880 -> maxim:MAX232
- IC4: value MEGA8-P -> 78L05Z; device atmel:MEGA8-P -> linear:78L05Z
- JP1: value RS232-USB -> Power; device jumper:JP4E -> jumper:JP1E
- JP2: value Reset -> 3V/5V; device jumper:JP1E -> jumper:JP2E
- JP3: value Power -> SDA
- JP5: value ISP -> Reset; device jumper:JP3Q -> jumper:JP1E
- R1, R2: value 4k7 -> see manual; device resistor:R-EU_0207/5V -> resistor:R-EU_R1206
- R10, R9: device resistor:R-EU_0207/5V -> resistor:R-EU_R1206
- R3: value 4k7 -> see manual; device resistor:R-EU_M1206 -> resistor:R-EU_R1206
- R4: value 10k -> see manual; device resistor:R-EU_0207/5V -> resistor:R-EU_R1206
- R7, R8: device resistor:R-EU_0207/5V -> resistor:R-EU_0309/V
Connections:
- removed net N$1: IC4.PD6(AIN0), R3.2
- removed net N$27: IC4.PD0(RXD), JP1.1
- removed net N$35: IC4.PD1(TXD), JP1.2
- removed net N$50: LED1.C, R3.1
- new net N$23: JP2.1, R5.1, R6.2
- new net N$34: C6.2, IC2G$1.C1-
- new net N$36: C6.1, IC2G$1.C1+
- new net N$37: IC3.VCCA, JP2.2, R1.1, R2.1
- new net N$38: C7.1, IC2G$1.C2+
- new net N$39: C7.2, IC2G$1.C2-
- new net N$40: IC2G$1.R2IN, X4.3
- new net N$41: IC3.SDAA, JP3.1, R1.2, SL2.3, SL3.3
- new net N$42: IC1.PC5(ADC5/SCL), IC3.SCLB, JP4.2, R4.2
- new net N$43: IC2G$1.T1OUT, X4.2
- new net N$45: C9.1, IC2G$1.V-
- new net N$46: C8.2, IC2G$1.V+
- new net RXD: IC1.PD0(RXD), IC2G$1.R2OUT, JP7.1
- new net TXD: IC1.PD1(TXD), IC2G$1.T1IN, JP7.2
- net GND: now also C13.2, C4.1, IC1.GND@1, IC2G$1.R1IN, IC2G$1.T2IN, IC2P.GND, IC3.GND, IC5.CS, IC5.VSS, JP5.2, JP6.6, JP7.3, R11.1, R6.1, SL2.1, SL3.1, SL4.1, X4.5; no longer C4.2, C6.1, IC2.CS, IC2.VSS, IC4.GND@1, JP1.3, JP2.2, JP5.6, R4.1, SL1.5, X2.1, X3.1
- net N$10: now also IC1.PC2(ADC2), IC5.Q2; no longer IC2.Q2, IC4.PC2(ADC2)
- net N$11: now also IC1.PC3(ADC3), IC5.Q1; no longer IC2.Q1, IC4.PC3(ADC3)
- net N$12: now also IC1.PD3(INT1), IC5.PHI2; no longer IC2.PHI2, IC4.PD3(INT1)
- net N$13: now also IC5.OSC1; no longer IC2.OSC1
- net N$14: now also IC5.OSC2; no longer IC2.OSC2
- net N$15: now also IC1.PB3(MOSI/OC2), JP6.4; no longer IC4.PB3(MOSI/OC2), JP5.4
- net N$16: now also IC5.IN+, IC5.VREF; no longer IC2.IN+, IC2.VREF
- net N$17: now also C12.1, SL4.3; no longer C7.1, SL1.1
- net N$18: now also IC1.PC6(/RESET), JP6.5; no longer IC4.PC6(/RESET), JP5.5
- net N$19: now also C4.2, IC1.PB7(XTAL2/TOSC2); no longer C5.2, IC4.PB7(XTAL2/TOSC2)
- net N$2: now also IC1.PD5(T1), IC5.RS0; no longer IC2.RS0, IC4.PD5(T1)
- net N$20: now also IC1.PB4(MISO), JP6.1; no longer IC4.PB4(MISO), JP5.1
- net N$21: now also C12.2; no longer C7.2
- net N$22: now also IC3.SCLA, JP4.1, SL2.2, SL3.2; no longer IC4.PC5(ADC5/SCL), X2.2, X3.2
- net N$24: now also IC5.IN-; no longer IC2.IN-
- net N$25: now also C11.2, IC5.ST/GT; no longer C8.2, IC2.ST/GT
- net N$26: now also C5.2, IC1.PB6(XTAL1/TOSC1); no longer C6.2, IC4.PB6(XTAL1/TOSC1)
- net N$28: now also IC1.PB5(SCK), JP6.3; no longer IC4.PB5(SCK), JP5.3
- net N$29: now also IC5.GS; no longer IC2.GS
- net N$3: now also IC1.PD4(XCK/T0), IC5.R/W; no longer IC2.R/W, IC4.PD4(XCK/T0)
- net N$30: now also C13.1, IC5.TONE, R11.2, SL4.2; no longer C9.1, IC2.TONE, R4.2, SL1.2
- net N$31: now also IC5.EST; no longer IC2.EST
- net N$32: now also C3.1, IC1.AREF; no longer C4.1, IC4.AREF
- net N$33: now also IC4.VI; no longer IC1.VI
- net N$4: now also IC1.PD2(INT0), IC5.IRQ/CP; no longer IC2.IRQ/CP, IC4.PD2(INT0)
- net N$5: now also IC1.PC4(ADC4/SDA), IC3.SDAB, JP3.2, R3.2; no longer IC4.PC4(ADC4/SDA), R1.2, X2.3, X3.3
- net N$58: now also C10.1, IC1.AVCC, IC1.VCC@1, JP1.1, JP6.2; no longer C3.1, IC4.AVCC, IC4.VCC@1, JP3.1, JP5.2
- net N$6: now also IC1.PD7(AIN1), JP5.1; no longer IC4.PD7(AIN1), JP2.1
- net N$8: now also IC1.PC0(ADC0), IC5.Q4; no longer IC2.Q4, IC4.PC0(ADC0)
- net N$9: now also IC1.PC1(ADC1), IC5.Q3; no longer IC2.Q3, IC4.PC1(ADC1)
- net VDD: now also C11.1, IC2P.VCC, IC3.EN, IC3.VCCB, IC4.VO, IC5.VDD, JP1.2, JP2.3, JP7.4, R3.1, R4.1, R5.2; no longer C10.1, IC1.VO, IC2.VDD, JP1.4, JP3.2, LED1.A, R1.1, R2.1
Other:
- moved on the sheet: C10, C3, C4, C5, C6, C7, C8, C9, JP3, R1, R2, R3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
