File: MYC_devices_hardware/MYCdevice_DTMF_Receiver/dtmf_rx.sch (EAGLE design)
At the start: 40 parts, among them IC1 MEGA8-P, IC2 MAX232, IC4 CM8870CP, IC5 78L05Z, Q1 20MHz, Q2 3,579545MHz, X1 8-15V, X2 1503_09, X3 1503_09, X4 RS232

Commit message: new board, bacom with includes
Parts:
- removed SL4: DTMF/RC5, con-amp-quick:M05
- removed X2, X3: 1503_09, con-lumberg:1503_09
- added IC3: PCA9517, PCA9517:PCA9517
- added JP5: Reset, jumper:JP1E
- added JP8: 5V, jumper:JP1E
- added R10: 10k, resistor:R-EU_R1206
- added R11: 4k7, resistor:R-EU_R1206
- added R2, R3: * see manual, resistor:R-EU_R1206
- added SL1, SL2: I2C, con-amp-quick:M03
- added SL3: DTMF, con-amp-quick:M03
- C1, C13, C14, C2, C3, C6: value 22uF 1210 -> 22uF
- C10, C7, C8, C9: value 22u 1210 -> 22uF
- IC4: value CM8870CP -> 78L05Z; device california-micro-devices:CM8870CP -> linear:78L05Z
- IC5: value 78L05Z -> CM8870CP; device linear:78L05Z -> california-micro-devices:CM8870CP
- JP2: value I2C -> 3V/5V; device jumper:JP1E -> jumper:JP2E
- JP3: value 5V -> SDA
- JP4: value Reset -> SCL
- R1: value 4k7 -> * see manual; device resistor:R-EU_0207/5V -> resistor:R-EU_R1206
- R4: value - -> * see manual; device resistor:R-EU_0207/5V -> resistor:R-EU_R1206
- R5: value 10k -> 1k; device resistor:R-EU_0207/5V -> resistor:R-EU_R1206
- R6: value 71,5k -> 1k5; device resistor:R-EU_0207/5V -> resistor:R-EU_R1206
- R7: device resistor:R-EU_0207/5V -> resistor:R-EU_R1206
- R8: value 4k7 -> 71,5k; device resistor:R-EU_0207/5V -> resistor:R-EU_R1206
- R9: value 4k7 -> -; device resistor:R-EU_0207/5V -> resistor:R-EU_R1206
- renumbered JP9 to JP7
Connections:
- removed net N$22: IC1.PC5(ADC5/SCL), JP2.2, R9.2, X2.2, X3.2
- new net N$10: JP2.1, R5.1, R6.2
- new net N$23: IC1.PC5(ADC5/SCL), IC3.SCLB, JP4.2, R4.2
- new net N$36: IC1.PC4(ADC4/SDA), IC3.SDAB, JP3.2, R3.2
- new net N$39: IC3.SCLA, JP4.1, R2.1, SL1.2, SL2.2
- new net N$43: IC3.VCCA, JP2.2, R1.2, R2.2
- net C13: now also C6.1; no longer C7.1
- net GND: now also C10.2, C9.1, IC3.GND, IC4.GND, IC5.INH, IC5.VSS, IC5.VSS@1, JP5.2, JP8.2, R6.1, SL1.1, SL2.1, SL3.1; no longer C10.1, C6.2, IC4.INH, IC4.VSS, IC4.VSS@1, IC5.GND, JP3.2, JP4.2, SL4.5, X2.1, X3.1
- net N$1: now also R11.2; no longer R1.2
- net N$13: now also C7.1; no longer C8.1
- net N$14: now also C6.2; no longer C7.2
- net N$16: now also C8.1; no longer C9.1
- net N$17: now also C9.2; no longer C10.2
- net N$21: now also SL3.3; no longer SL4.1
- net N$24: now also R10.1; no longer R5.1
- net N$25: now also IC5.IN-, R10.2, R8.2, R9.2; no longer IC4.IN-, R4.2, R5.2, R6.2
- net N$26: now also IC5.GS, R8.1, R9.1; no longer IC4.GS, R4.1, R6.1
- net N$29: now also IC5.OSC2; no longer IC4.OSC2
- net N$3: now also C7.2; no longer C8.2
- net N$30: now also IC5.Q3; no longer IC4.Q3
- net N$31: now also IC5.OSC1; no longer IC4.OSC1
- net N$32: now also IC5.EST; no longer IC4.EST
- net N$33: now also IC4.VI; no longer IC5.VI
- net N$34: now also IC5.Q1; no longer IC4.Q1
- net N$38: now also IC5.Q2; no longer IC4.Q2
- net N$40: now also IC5.ST/GT; no longer IC4.ST/GT
- net N$42: now also IC5.STD; no longer IC4.STD
- net N$44: now also C10.1; no longer C6.1
- net N$5: now also IC3.SDAA, JP3.1, R1.1, SL1.3, SL2.3; no longer IC1.PC4(ADC4/SDA), JP2.1, R8.2, X2.3, X3.3
- net N$50: now also R11.1; no longer R1.1
- net N$6: now also JP5.1; no longer JP4.1
- net N$7: now also IC5.IN+, IC5.VREF; no longer IC4.IN+, IC4.VREF
- net N$8: now also IC5.Q4; no longer IC4.Q4
- net VDD: now also C8.2, IC3.EN, IC3.VCCB, IC4.VO, IC5.TOE, IC5.VDD, JP2.3, JP8.1, R3.1, R4.1, R5.2; no longer C9.2, IC4.TOE, IC4.VDD, IC5.VO, JP3.1, R8.1, R9.1
Other:
- moved on the sheet: C10, C6, C7, C8, C9, JP3, JP4, R1, R4, R5, R6, R8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
