File: MYC_devices_hardware/MYCdevice_create_rotator_control/rotorsteuerung_create.sch (EAGLE design)
At the start: 52 parts, among them IC1 MEGA8-P, IC3 7805T, K1 RT424012, K2 RT424012, K3 RT424012, Q1 20MHz, T1 BC547, T2 BC547, T3 BC547

Commit message: new board. firmware with correction of nonlinearity and other
Parts:
- removed C13, C14, C15: 22u, resistor:C-EUC1206
- removed IC3: 7805T, linear:7805T
- removed JP3: Power, jumper:JP1E
- removed R12: 15k 1%, rcl:R-EU_0204/7
- removed R13, R16, R18: 82k, rcl:R-EU_0204/7
- removed R14: 7,5, rcl:R-EU_0204/7
- removed R15: 47, rcl:R-EU_0204/7
- removed R17, R19: 47k, rcl:R-EU_0204/7
- removed R20: 220k, rcl:R-EU_0204/7
- removed SL5: Motor, con-amp-quick:M05
- added C2, C3: 22u, resistor:C-EUC1206
- added C5, C6: 18pF, resistor:C-EU050-025X075
- added D7: 1N4004, zetex:D_E2L
- added IC2: 78L05, v-reg:78LXX
- added JP4: USB, jumper:JP4E
- added R2: 4k7, resistor:R-EU_0204/2V
- added R4: 3.3k, resistor:R-EU_0204/2V
- added R6: Ry, rcl:R-EU_0204/7
- added SL1: I2C, con-amp-quick:M05
- C1: value 22u -> 1000u16V; device resistor:C-EUC1206 -> rcl:CPOL-EUE5-10.5
- C7, C8: value 18pF -> 22u; device resistor:C-EU050-025X075 -> resistor:C-EUC1206
- R1: value 3.3k -> 4k7
- R10: value 10k 1% -> 220k
- R11: value 1000M -> 220k
- R7, R8: value 4k7 -> Ry; device resistor:R-EU_0204/2V -> rcl:R-EU_0204/7
- R9: value 220k -> 75k
- SL2: value I2C -> Poti
- SL3: value Poti -> Motor
Connections:
- removed net N$11: K12.P, SL5.4
- removed net N$18: K22.P, K32.P, SL5.1
- removed net N$21: C15.1, D5.C, D6.A, IC1.PC1(ADC1), R10.1, R11.1, R12.1, R13.1, R14.1, R15.1, R20.1, R9.1
- removed net N$24: C1.1, D1.C, D2.C, D3.C, D4.A, IC3.VI, K11.2, K21.2, K31.2
- removed net N$27: C12.2, R14.2, R15.2, R16.2, SL3.3, VR1.C
- removed net N$29: IC1.AVCC, IC1.VCC@1, JP3.1
- removed net N$39: R16.1, R17.2, VR1.R
- removed net N$44: R18.1, R19.2, VR2.R
- new net C7: C7.2, D7.C, OK1.A, SL2.4
- new net C9: C9.2, R10.2, SL2.3, VR1.C, VR1.R
- new net CCW: K13.O, SL3.2
- new net CW: K12.O, SL3.5
- new net N$30: IC1.PD0(RXD), JP4.1
- new net N$32: IC1.PD1(TXD), JP4.2
- new net TO1: K22.P, K32.P, SL3.1
- new net TO2: K12.P, SL3.4
- new net TO3: K13.P, SL3.3
- net GND: now also C1.-, C12.2, C2.2, C3.2, C4.1, C5.1, C6.1, IC2.GND, JP4.3, R7.1, R8.1, SL1.1, SL1.3, VR2.R; no longer C1.2, C12.1, C13.1, C14.1, C15.2, C4.2, IC3.GND, R17.1, R18.2, R20.2, R9.2, SL2.1, SL2.3
- net N$1: now also R1.2, SL1.5; no longer R7.2, SL2.5
- net N$10: now also R10.1, R11.1, R9.1; no longer K13.O, SL5.2
- net N$13: now also R4.1; no longer R3.1
- net N$17: now also C12.1, D5.C, D6.A, IC1.PC1(ADC1), R6.2, R8.2, R9.2; no longer K12.O, SL5.5
- net N$19: now also C5.2; no longer C8.2
- net N$2: now also C1.+, C2.1, D4.C, IC2.IN; no longer K13.P, SL5.3
- net N$22: now also R4.2; no longer R3.2
- net N$25: now also D1.C, D2.C, D3.C, D4.A, K11.2, K21.2, K31.2, SL1.2; no longer D4.C, SL2.2
- net N$28: now also C10.2, SL2.2; no longer C13.2, R10.2, SL3.2
- net N$3: now also C8.2, D7.A, SL2.5; no longer C11.2, SL3.5
- net N$33: now also R3.1; no longer R1.1
- net N$34: now also R3.2; no longer R1.2
- net N$35: now also C4.2; no longer C9.2
- net N$37: now also C6.2; no longer C7.2
- net N$4: now also C11.2, SL2.1; no longer C14.2, R12.2, R13.2, R19.1, SL3.1
- net N$5: now also R2.2, SL1.4; no longer R8.2, SL2.4
- net N$7: now also R6.1, R7.2; no longer C10.2, OK1.A, SL3.4
- net VDD: now also C3.1, IC1.AVCC, IC1.VCC@1, IC2.OUT, JP4.4, R1.1, R2.1; no longer C4.1, IC3.VO, JP3.2, R7.1, R8.1
Other:
- moved on the sheet: C10, C11, C12, C4, C7, C8, C9, D4, R1, R10, R11, R3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

Commit message: new board and slavecore1.7
Parts:
- added IC3: PCA9517, PCA9517:PCA9517
- added JP3: SDA, jumper:JP1E
- added JP5: Reset, jumper:JP1E
- added JP6: ISP, jumper:JP3Q
- added JP7: USB, jumper:JP4E
- added R12: 220k, rcl:R-EU_0204/7
- added R31, R41, R51: 3.3k, resistor:R-EU_R1206
- C1: value 1000u16V -> 22u; device rcl:CPOL-EUE5-10.5 -> resistor:C-EUC1206
- C4: value 22u -> 18pF; device resistor:C-EUC1206 -> resistor:C-EU025-024X044
- C5: device resistor:C-EU050-025X075 -> resistor:C-EU025-024X044
- C6: value 18pF -> 470u16V; device resistor:C-EU050-025X075 -> rcl:CPOL-EUE5-10.5
- IC1: value MEGA8-P -> MEGA8-AI; device atmel:MEGA8-P -> atmel:MEGA8-AI
- JP1: value Reset -> Power
- JP2: value ISP -> 3,3V/5V; device jumper:JP3Q -> jumper:JP2E
- JP4: value USB -> SCL; device jumper:JP4E -> jumper:JP1E
- R1, R2: value 4k7 -> see manual; device resistor:R-EU_0204/2V -> resistor:R-EU_M1206
- R10: value 220k -> 75k
- R3, R4: value 3.3k -> see manual; device resistor:R-EU_0204/2V -> resistor:R-EU_R1206
- R5: value 3.3k -> 1k; device resistor:R-EU_0204/2V -> resistor:R-EU_R1206
- R6: value Ry -> 1k5; device rcl:R-EU_0204/7 -> resistor:R-EU_R1206
- R9: value 75k -> Ry
- T1, T2, T3: value BC547 -> (none); device transistor:BC547 -> transistor:BC817-16-NPN-SOT23-BEC
- renumbered IC2 to IC4
Connections:
- removed net N$2: C1.+, C2.1, D4.C, IC4.IN
- new net N$11: IC1.AVCC, IC1.VCC@1, IC1.VCC@2, JP1.1, JP6.2
- new net N$18: JP2.1, R5.1, R6.2
- new net N$24: IC3.SDAA, JP3.1, R1.2, SL1.5
- new net N$27: IC3.SCLA, JP4.1, R2.2, SL1.4
- new net N$29: IC3.VCCA, JP2.2, R1.1, R2.1
- new net N$44: IC1.PC5(ADC5/SCL), IC3.SCLB, JP4.2, R3.2
- net C9: now also R11.2; no longer R10.2
- net GND: now also C1.2, C3.1, C6.-, IC1.GND@2, IC3.GND, JP5.1, JP6.6, JP7.3, R6.1, R9.1; no longer C1.-, C3.2, C6.1, JP1.1, JP2.6, JP4.3, R7.1
- net N$1: now also IC3.SDAB, JP3.2, R4.2; no longer R1.2, SL1.5
- net N$10: now also R12.1; no longer R9.1
- net N$13: now also R41.1; no longer R4.1
- net N$15: now also IC1.PD4(XCK/T0), R51.1; no longer IC1.PB2(SS/OC1B), R5.1
- net N$17: now also R10.2, R7.2; no longer R6.2, R8.2
- net N$19: now also C4.2; no longer C5.2
- net N$20: now also JP6.3; no longer JP2.3
- net N$22: now also IC1.PD3(INT1), R41.2; no longer IC1.PB1(OC1A), R4.2
- net N$25: now also C1.1, C6.+, D4.C, IC4.IN; no longer D4.A, SL1.2
- net N$26: now also JP5.2; no longer JP1.2
- net N$28: now also R12.2; no longer R11.2
- net N$30: now also JP7.1; no longer JP4.1
- net N$31: now also JP6.4; no longer JP2.4
- net N$32: now also JP7.2; no longer JP4.2
- net N$33: now also IC1.PD2(INT0), R31.1; no longer IC1.PB0(ICP), R3.1
- net N$34: now also R31.2; no longer R3.2
- net N$35: now also C3.2; no longer C4.2
- net N$36: now also R51.2; no longer R5.2
- net N$37: now also C5.2; no longer C6.2
- net N$38: now also JP6.5; no longer JP2.5
- net N$5: now also D4.A, SL1.2; no longer IC1.PC5(ADC5/SCL), R2.2, SL1.4
- net N$7: now also R7.1, R8.2; no longer R6.1, R7.2
- net N$8: now also JP6.1; no longer JP2.1
- net VDD: now also C2.1, IC3.EN, IC3.VCCB, JP1.2, JP2.3, JP7.4, R3.1, R4.1, R5.2; no longer C3.1, IC1.AVCC, IC1.VCC@1, JP2.2, JP4.4, R1.1, R2.1
Other:
- moved on the sheet: C2, C3, C4, C5, D4, JP1, R1, R10, R11, R2, R3, R4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
