File: MYC_devices_hardware/MYCdevice_voice_output/spachausgabe.sch (EAGLE design)
At the start: 48 parts, among them IC1 MEGA8-P, IC2 MAX232, IC3 7805TV, Q1 20MHz, X1 8-15V, X2 1503_09, X3 1503_09, X4 RS232, X5 1503_09

Commit message: new board (MSM4); bascom with include files
Parts:
- removed JP13: Modul2, jumper:JP3QE
- removed OK1, OK10, OK2, OK3, OK4, OK5, OK6, OK7, OK8, OK9: CNY17, optocoupler:CNY17
- removed R10, R11, R12, R7, R8, R9: 1k, resistor:R-EU_M1206
- removed X2, X3: 1503_09, con-lumberg:1503_09
- added IC4: 78L05Z, linear:78L05Z
- added JP2: 3V/5V, jumper:JP2E
- added JP3: SDA, jumper:JP1E
- added JP5: Reset, jumper:JP1E
- added JP7: US7, jumper:JP4E
- added SL1, SL2: (no value), con-amp-quick:M03
- C1, C2, C3, C6: value 22uF 1210 -> 22uF
- C10, C7, C8, C9: value 22u 1210 -> 22uF
- IC1: value MEGA8-P -> MEGA8-AI; device atmel:MEGA8-P -> atmel:MEGA8-AI
- IC3: value 7805TV -> PCA9517; device linear:7805TV -> PCA9517:PCA9517
- JP4: value Reset -> SCL
- JP9: value USB -> Modul2; device jumper:JP4E -> jumper:JP3QE
- R1: value 4k7 -> see manual; device resistor:R-EU_0207/5V -> resistor:R-EU_R1206
- R2: value 4k7 -> see manual; device resistor:R-EU_0207/5V -> resistor:R-EU_M1206
- R3, R4: value 1k -> see manual; device resistor:R-EU_M1206 -> resistor:R-EU_R1206
- R5: device resistor:R-EU_M1206 -> resistor:R-EU_R1206
- R6: value 1k -> 1k5; device resistor:R-EU_M1206 -> resistor:R-EU_R1206
- renumbered JP12 to JP8
Connections:
- removed net N$24: JP8-9.2, OK8.EMI
- removed net N$29 (its old number): JP8-8.2, OK7.EMI
- removed net N$31: JP8-9.1, OK8.COL
- removed net N$32: JP8-5.1, OK4.COL
- removed net N$36: JP8-3.1, OK2.COL
- removed net N$38: JP13-1.1, OK10.COL
- removed net N$40: JP8-10.1, OK9.COL
- removed net N$41: JP8-3.2, OK2.EMI
- removed net N$42: JP8-8.1, OK7.COL
- removed net N$43: JP8-4.1, OK3.COL
- removed net N$45: JP8-4.2, OK3.EMI
- removed net N$46: JP8-5.2, OK4.EMI
- removed net N$47: JP8-6.1, OK5.COL
- removed net N$48: JP8-6.2, OK5.EMI
- removed net N$49: OK9.C, R11.2
- removed net N$50: OK8.C, R10.2
- removed net N$53: JP8-7.1, OK6.COL
- removed net N$54: JP8-7.2, OK6.EMI
- removed net N$55: JP8-2.1, OK1.COL
- removed net N$56: JP8-2.2, OK1.EMI
- removed net N$57: OK7.C, R9.2
- removed net N$58: OK6.C, R8.2
- removed net N$59: OK5.C, R7.2
- removed net N$62: OK4.C, R6.2
- removed net N$64: OK2.C, R4.2
- removed net N$65: OK1.C, R3.2
- net C13: now also C6.1; no longer C7.1
- net GND: now also C10.2, C9.1, IC1.GND@2, IC4.GND, JP5.2, JP7.3, JP8-10.2, JP8-2.2, JP8-3.2, JP8-4.2, JP8-5.2, JP8-6.2, JP8-7.2, JP8-8.2, JP8-9.2, JP9-1.2, JP9-2.1, JP9-2.2, JP9-3.2, R6.1, SL1.1, SL2.1; no longer C10.1, C6.2, JP13-2.1, JP13-2.2, JP13-3.2, JP4.2, JP9.3, X2.1, X3.1
- net N$1: now also JP8-10.1; no longer R11.1
- net N$10: now also IC3.SCLA, JP4.1, R2.2, SL1.2, SL2.2; no longer OK3.C, R5.2
- net N$11: now also IC3.VCCA, JP2.2, R1.1, R2.1; no longer OK10.C, R12.2
- net N$12: now also JP7.2; no longer JP9.2
- net N$13: now also C7.1; no longer C8.1
- net N$14: now also C6.2; no longer C7.2
- net N$16: now also C8.1; no longer C9.1
- net N$17: now also C9.2; no longer C10.2
- net N$2: now also JP7.1; no longer JP9.1
- net N$21: now also JP2.1, R5.1, R6.2; no longer JP8-10.2, OK9.EMI
- net N$22: now also IC3.SCLB, JP4.2, R4.2; no longer R2.2, X2.2, X3.2
- net N$23: now also JP8-8.1; no longer R9.1
- net N$25: now also JP8-3.1; no longer R4.1
- net N$26: now also JP8-4.1; no longer R5.1
- net N$3: now also C7.2; no longer C8.2
- net N$30: now also JP9-1.1; no longer R12.1
- net N$33: now also IC4.VI; no longer IC3.VI
- net N$34: now also JP8-2.1; no longer R3.1
- net N$39: now also JP8-5.1; no longer R6.1
- net N$44: now also C10.1, IC1.VCC@2; no longer C6.1
- net N$5: now also IC3.SDAB, JP3.2, R3.2; no longer R1.2, X2.3, X3.3
- net N$51: now also JP8-7.1; no longer R8.1
- net N$52: now also JP8-6.1; no longer R7.1
- net N$6: now also JP5.1; no longer JP4.1
- net N$7: now also JP8-9.1; no longer R10.1
- net N$8: now also IC3.SDAA, JP3.1, R1.2, SL1.3, SL2.3; no longer JP13-1.2, OK10.EMI
- net VDD: now also C8.2, IC3.EN, IC3.VCCB, IC4.VO, JP2.3, JP7.4, JP9-3.1, R3.1, R4.1, R5.2; no longer C9.2, IC3.VO, JP13-3.1, JP9.4, OK1.A, OK10.A, OK2.A, OK3.A, OK4.A, OK5.A, OK6.A, OK7.A, OK8.A, OK9.A, R1.1, R2.1
Other:
- moved on the sheet: C10, C6, C7, C8, C9, D1, JP4, JP6, R1, R2, R3, R4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
