File: MYC_devices_hardware/MYCdevice_electronic_load/electronic_load.sch (EAGLE design)
At the start: 118 parts, among them IC1 ATMEGA644A, IC10 MCP4921, IC11 LM324N, IC12 LM324N, IC13 79L09, IC14 MCP4921, IC2 MAX232, IC21 MCP60x4, IC22 MCP60x4, IC3 PCA9517, IC4 78L5, IC5 MCP4921, IC6 MCP4921, IC7 MCP4921, IC8 MCP4921, IC9 MCP4921, Q1 20MHz, T1 BC807, T2 BC817, X1 8-15V, X4 RS232

Commit message: board with 16bit AD + corresponding firmware + doc
Parts:
- removed C244: 18pF, resistor:C-EU025-025X050
- removed IC1: ATMEGA644A, atmel:ATMEGA644A
- removed IC21, IC22: MCP60x4, linear:LM324D
- removed JP11, JP12: (no value), jumper:JP4E
- removed R41, R43, R45, R47, R49, R51: 154k, resistor:R-EU_M1206
- removed R42, R44, R46, R48, R50, R52: 18k, resistor:R-EU_M1206
- removed R53: 180, resistor:R-EU_R1206
- removed R54: 1k5, resistor:R-EU_R1206
- added C23, C24, C25, C26, C29, C30, C31, C32, C35, C36, C37, C38, C41, C42: 22n, resistor:C-EUC1206
- added C27, C28, C33, C34, C39, C40, C43: 220n, resistor:C-EUC1206
- added C50, C51: 22uF, rcl:C-EUC1206
- added IC15: MEGA8-AI, atmel:MEGA8-AI
- added R12: 100, resistor:R-EU_R1206
- added SL10, SL9: Iin, con-amp-quick:M05
- added SL11: U/Iin, con-amp-quick:M05
- added SL3: Gates1, con-amp-quick:M05
- C4: value 22uF -> 18pF; device rcl:C-EUC1206 -> resistor:C-EU025-025X050
- JP10: value (none) -> ISP
- R25, R27, R29, R33, R35, R37: value 154k -> 100; device resistor:R-EU_M1206 -> resistor:R-EU_R1206
- R26, R30, R32, R34, R36: value 18k -> 100; device resistor:R-EU_M1206 -> resistor:R-EU_R1206
- R28: value 18k -> 100
- R31: value 154 -> 100; device resistor:R-EU_M1206 -> resistor:R-EU_R1206
- R38: value 18k -> see maunual; device resistor:R-EU_M1206 -> resistor:R-EU_R1206
- R39: value 154k -> see manual; device resistor:R-EU_M1206 -> resistor:R-EU_R1206
- R40: value 18k -> 2k2; device resistor:R-EU_M1206 -> resistor:R-EU_R1206
- SL4: value Iin -> Gates2
- SL5: value Iin -> AD_F1_U; device con-amp-quick:M05 -> con-amp-quick:M10
- SL6: value U/Iin -> AD_F3_F2; device con-amp-quick:M05 -> con-amp-quick:M10
- SL7: value Gates1 -> AD_F5_F4; device con-amp-quick:M05 -> con-amp-quick:M10
- SL8: value Gates2 -> ADF7_F6; device con-amp-quick:M05 -> con-amp-quick:M10
Connections:
- removed net I1: IC1.(PCINT1/ADC1)PA1, IC21A.OUT, JP12.1, R25.2
- removed net I2: IC1.(PCINT2/ADC2)PA2, IC21B.OUT, JP12.2, R29.2
- removed net I3: IC1.(PCINT3/ADC3)PA3, IC21D.OUT, JP12.3, R33.2
- removed net I4: IC1.(PCINT4/ADC4)PA4, IC21C.OUT, JP12.4, R37.2
- removed net I5: IC1.(PCINT5/ADC5)PA5, IC22A.OUT, JP11.1, R41.2
- removed net I6: IC1.(PCINT6/ADC6)PA6, IC22D.OUT, JP11.2, R45.2
- removed net I7: IC1.(PCINT7/ADC7)PA7, IC22C.OUT, JP11.3, R49.2
- removed net N$2: IC1.(PCINT24/RXD0)PD0, IC2G$1.R1OUT, JP7.1
- removed net N$25: C3.2, IC1.AREF
- removed net N$34: IC22D.-IN, R45.1, R46.1
- removed net N$41: IC21D.-IN, R33.1, R34.1
- removed net N$44: IC21C.+IN, R39.1, R40.2
- removed net N$47: IC22A.-IN, R41.1, R42.1
- removed net N$52: R48.1, SL6.1
- removed net N$53: R46.2, SL6.2
- removed net N$65: R28.1, SL4.1
- removed net N$66: R32.1, SL4.3
- removed net N$67: IC21A.+IN, R27.1, R28.2
- removed net N$68: R36.2, SL4.5
- removed net N$69: R26.2, SL4.2
- removed net N$79: R34.2, SL5.1
- removed net N$80: IC21D.+IN, R35.1, R36.1
- removed net N$89: R50.2, SL6.4
- removed net N$90: IC22C.+IN, R51.1, R52.2
- new net I1N: R37.1, SL11.4
- new net I1P: R36.1, SL11.3
- new net I2N: R35.1, SL11.2
- new net I2P: R34.1, SL11.1
- new net I3N: R33.1, SL10.5
- new net I3P: R32.1, SL10.4
- new net I4N: R31.1, SL10.3
- new net I4P: R30.1, SL10.2
- new net I5N: R29.1, SL10.1
- new net I5P: R28.1, SL9.5
- new net I6N: R27.1, SL9.4
- new net I6P: R26.1, SL9.3
- new net I7N: R25.1, SL9.2
- new net I7P: R12.1, SL9.1
- new net N$71: C25.2, C27.2, R25.2, SL8.3
- new net N$78: C41.2, C43.1, R37.2, SL5.3
- new net SCL2: IC15.PD7(AIN1), SL5.8, SL6.6, SL6.8, SL7.8, SL8.8
- new net SDA2: IC15.PD6(AIN0), SL5.6, SL5.7, SL6.7, SL7.7, SL8.7
- net FET1: now also IC10A.CS, IC15.PD4(XCK/T0); no longer IC1.(PCINT20/TDO)PC4, IC7A.CS
- net FET2: now also IC15.PD3(INT1), IC9A.CS; no longer IC1.(PCINT23/TOSC2)PC7, IC14A.CS
- net FET3: now also IC15.PD2(INT0), IC8A.CS; no longer IC1.(PCINT21/TDI)PC5, IC6A.CS
- net FET4: now also IC15.PC3(ADC3), IC7A.CS; no longer IC1.(PCINT22/TOSC1)PC6, IC5A.CS
- net FET5: now also IC15.PC2(ADC2), IC6A.CS; no longer IC1.(PCINT18/TCK)PC2, IC9A.CS
- net FET6: now also IC15.PC1(ADC1), IC5A.CS; no longer IC1.(PCINT19/TMS)PC3, IC8A.CS
- net FET7: now also IC14A.CS, IC15.PC0(ADC0); no longer IC1.(PCINT31/OC2A)PD7, IC10A.CS
- net GND: now also C23.1, C24.1, C25.1, C26.1, C29.1, C30.1, C31.1, C32.1, C35.1, C36.1, C37.1, C38.1, C4.1, C41.1, C42.1, C50.2, C51.1, IC15.GND, IC15.GND@1, IC15.GND@2, R38.2, SL3.5, SL4.4, SL4.5, SL5.1, SL5.9, SL6.9, SL7.6, SL7.9, SL8.9; no longer C244.1, C4.2, IC1.GND, IC1.GND@1, IC1.GND@2, IC1.GND@3, IC21P.V-, IC22B.+IN, IC22P.V-, R27.2, R31.2, R35.2, R43.2, R47.2, R51.2, R54.2, SL7.5, SL8.4, SL8.5
- net GON: now also IC15.PB0(ICP); no longer IC1.(PCINT29/OC1A)PD5
- net LDAC: now also IC15.PD5(T1); no longer IC1.(PCINT30/OC2B/ICP)PD6
- net N$1: now also C26.2, C27.1, R12.2, SL8.4; no longer IC21A.-IN, R25.1, R26.1
- net N$11: now also IC15.PB7(XTAL2/TOSC2); no longer IC1.XTAL1
- net N$15: now also IC15.PB4(MISO); no longer IC1.(PCINT14/MISO)PB6
- net N$18: now also IC15.PC6(/RESET); no longer IC1.RESET
- net N$19: now also C4.2, IC15.PB6(XTAL1/TOSC1); no longer C244.2, IC1.XTAL2
- net N$21: now also IC14A.VOUT; no longer IC7A.VOUT
- net N$23: now also IC15.PB3(MOSI/OC2); no longer IC1.(PCINT13/MOSI)PB5
- net N$24: now also IC9A.VOUT; no longer IC8A.VOUT
- net N$26: now also IC8A.VOUT; no longer IC9A.VOUT
- net N$27: now also R40.2, SL11.5; no longer R53.2, SL6.5
- net N$29: now also C31.2, C33.1, R29.2, SL7.3; no longer R30.2, SL4.4
- net N$30: now also C30.2, C34.2, R30.2, SL7.2; no longer IC21B.-IN, R29.1, R30.1
- net N$31: now also IC5A.VOUT; no longer IC14A.VOUT
- net N$32: now also C29.2, C34.1, R31.2, SL7.1; no longer IC22C.-IN, R49.1, R50.1
- net N$35: now also IC15.PC4(ADC4/SDA); no longer IC1.(PCINT17/SDA)PC1
- net N$37: now also IC15.PB2(SS/OC1B); no longer IC1.(PCINT12/OC0B/!SS!)PB4
- net N$4: now also C50.1, C51.2, IC15.AVCC, IC15.VCC@1, IC15.VCC@2; no longer C4.1, IC1.AVCC, IC1.VCC, IC1.VCC@1, IC1.VCC@2
- net N$42: now also IC15.PD0(RXD), IC2G$1.R1OUT, JP7.1; no longer IC1.(PCINT8/XCK0/T0)PB0, R11.1
- net N$45: now also C38.2, C39.2, R32.2, SL6.4; no longer IC21C.-IN, R37.1, R38.1
- net N$46: now also IC15.PB5(SCK); no longer IC1.(PCINT15/SCK)PB7
- net N$48: now also C37.2, C39.1, R33.2, SL6.3; no longer R44.1, SL5.4
- net N$49: now also C36.2, C40.2, R34.2, SL6.2; no longer IC21B.+IN, R31.1, R32.2
- net N$50: now also IC15.PC5(ADC5/SCL); no longer IC1.(PCINT16/SCL)PC0
- net N$54: now also IC15.PB1(OC1A), R11.1; no longer R38.2, SL5.3
- net N$55: now also IC7A.VOUT; no longer IC5A.VOUT
- net N$6: now also IC15.PD1(TXD); no longer IC1.(PCINT25/TXD0)PD1
- net N$60: now also C3.2, IC15.AREF; no longer R42.2, SL5.5
- net N$70: now also C24.2, C28.1, R26.2, SL8.2; no longer R40.1, SL5.2
- net N$72: now also C35.2, C40.1, R35.2, SL6.1; no longer IC22A.+IN, R43.1, R44.2
- net N$74: now also C23.2, C28.2, R27.2, SL8.1; no longer IC22D.+IN, R47.1, R48.2
- net N$76: now also C42.2, C43.2, R36.2, SL5.4; no longer R52.1, SL6.3
- net N$8: now also C32.2, C33.2, R28.2, SL7.4; no longer IC22B.-IN, IC22B.OUT
- net SFET1: now also IC12C.OUT, R24.2, SL4.3; no longer IC11D.OUT, R18.2, SL7.1
- net SFET2: now also IC12A.OUT, R20.2, SL4.2; no longer IC11A.OUT, R14.2, SL7.2
- net SFET3: now also IC12D.OUT, R22.2, SL4.1; no longer IC11C.OUT, R16.2, SL7.3
- net SFET4: now also SL3.4; no longer SL7.4
- net SFET5: now also IC11C.OUT, R16.2, SL3.3; no longer IC12D.OUT, R22.2, SL8.1
- net SFET6: now also IC11A.OUT, R14.2, SL3.2; no longer IC12A.OUT, R20.2, SL8.2
- net SFET7: now also IC11D.OUT, R18.2, SL3.1; no longer IC12C.OUT, R24.2, SL8.3
- net U: now also R38.1, R39.1, R40.1, SL5.2; no longer IC1.(PCINT0/ADC0)PA0, R53.1, R54.1
- net VDD: now also SL5.10, SL6.10, SL7.10, SL8.10, SL8.6; no longer IC21P.V+, IC22P.V+
Other:
- note added: "33k extern for 90V"
- note removed: "+ extern 51k for 90V"
