File: MYC_devices_hardware/V_I_sensor/U_I.sch (EAGLE design)
At the start: 35 parts, among them IC2 MEGA8-AI, IC3 78L05, IC4 MAX3232CSE, Q1 20MH2, U1 INA219AIDCNR, X1 8-15V, X4 RS232

Commit message: reduced board!
Parts:
- removed C1, C2: 22uF, rcl:C-EUC1206
- removed C6, C7, C8, C9: 220n, rcl:C-EUC1206
- removed D1: 1N4004, diode:1N4004
- removed IC3: 78L05, v-reg:78LXX
- removed IC4: MAX3232CSE, maxim:MAX3232CSE
- removed JP10, JP9: wireless, jumper:JP4E
- removed JP12: no_remote, jumper:JP1E
- removed X1: 8-15V, con-conrad:737992-55
- removed X4: RS232, con-subd:F09H
- added JP8: INA219, jumper:JP4E
- R4, R5: value 10 -> 10k
Connections:
- removed net C13: C6.1, IC4G$1.C1+
- removed net CLK0: IC2.PC2(ADC2), JP10.4
- removed net GPIO1: IC2.PC1(ADC1), JP10.2
- removed net N$10: IC4G$1.T1OUT, X4.2
- removed net N$13: C7.1, IC4G$1.C2+
- removed net N$14: C6.2, IC4G$1.C1-
- removed net N$16: C8.1, IC4G$1.V+
- removed net N$17: C9.2, IC4G$1.V-
- removed net N$20: IC2.PB0(ICP), JP12.1
- removed net N$27: D1.A, X1.-1
- removed net N$3: C7.2, IC4G$1.C2-
- removed net N$33: C1.1, D1.C, IC3.IN
- removed net N$41: IC4G$1.R2IN, X4.3
- removed net SCS: IC2.PC0(ADC0), JP9.3
- net GND: no longer C1.2, C2.2, C9.1, IC3.GND, IC4G$1.R1IN, IC4G$1.T2IN, IC4P.GND, JP12.2, JP9.2, X1.+, X1.K, X4.5
- net N$12: no longer IC4G$1.T1IN
- net N$2: no longer IC4G$1.R2OUT
- net N$22: now also JP8.1
- net N$26: no longer JP9.4
- net N$4: no longer JP10.3
- net N$5: now also JP8.2
- net N$9: no longer JP10.1
- net VDD: now also JP8.3; no longer C2.1, C8.2, IC3.OUT, IC4P.VCC, JP9.1
Other:
- note added: "connect on wirelayer side!"
