File: MYC_devices_hardware/wireless_interface/wireless_interface.sch (EAGLE design)
At the start: 41 parts, among them IC1 ATMEGA644A, IC2 7805DT, IC3 PCA9517, IC4 MAX3232CSE, Q1 20MH

Commit message: new bord and firmware with Lora and 2.4GHz
Parts:
- removed DC1: 12V - 3V, dc-dc-converter:NME
- removed SV1: wireless modul, con-amp-mt:S12P
- added C13, C14: 22uF, rcl:C-EUC1206
- added IC5: 7803, linear:7805TV
- added J1: 1050171001, 1050171001:1050171001
- added JP10: Power, jumper:JP2E
- added JP16: nRF24L1 WLAN, jumper:JP4E
- added JP17, JP18: nRF24L1s, jumper:JP4E
- added JP20: Bluetooth, jumper:JP4E
- added JP35: JP35, jumper:JP2E
- added JP36: JP36, jumper:JP2E
- added JP37: Sensor, jumper:JP4E
- added JP39, JP40: GPS, jumper:JP4E
- added JP41: Light Klima, jumper:JP4E
- added JP9: RS232, jumper:JP2E
- added PAD1: Pad1, wirepad:WIREPADSMD1,27-254
- added U1: TXS0108EPWRG4, TXS0108EPWRG4:TXS0108EPWRG4
- JP12: value RS232 -> RFM95
- JP13: value JP13 -> RFM95
- JP14: value JP14 -> RFM95
- JP15: value 9-12V -> nRF24L1WLAN; device jumper:JP1E -> jumper:JP4E
- JP19: value Light Klima -> nRF24L1s
- JP21: value Sensor -> Bluetooth
- renumbered JP22 to JP38
Connections:
- removed net N$31: D1.A, JP15.2
- removed net RESET_W: IC1.(PCINT23/TOSC2)PC7, SV1-3.S
- removed net X1: IC1.(PCINT9/CLKO/T1)PB1, SV1-4.S
- removed net X2: IC1.(PCINT8/XCK0/T0)PB0, SV1-5.S
- removed net X3: IC1.(PCINT22/TOSC1)PC6, SV1-6.S
- removed net X4: IC1.(PCINT21/TDI)PC5, SV1-12.S
- new net B_MOD: IC1.(PCINT0/ADC0)PA0, JP20.1
- new net COM2_RX*: JP20.3, U1.A6
- new net COM2_TX_50HZ*: PAD1.P, U1.A5
- new net GEN: IC1.(PCINT31/OC2A)PD7, JP39.1
- new net GFIX: IC1.(PCINT30/OC2B/ICP)PD6, JP39.3
- new net GPPS: IC1.(PCINT29/OC1A)PD5, JP40.4
- new net INT/G0*: JP13.1, U1.A7
- new net INT_G0: IC1.(PCINT9/CLKO/T1)PB1, U1.B7
- new net MISO: IC1.(PCINT14/MISO)PB6, JP6.1, U1.B4
- new net MOSI: IC1.(PCINT13/MOSI)PB5, JP14.1, JP6.4, U1.B1
- new net N$11: D1.A, JP10.2
- new net RESET/CE*: JP15.2, JP17.4, U1.A8
- new net RESET_CE: IC1.(PCINT23/TOSC2)PC7, JP14.3, U1.B8
- new net SCK: IC1.(PCINT15/SCK)PB7, JP13.2, JP6.3, U1.B3
- new net SCS: IC1.(PCINT12/OC0B/!SS!)PB4, JP14.2, U1.B2
- net COM2_RX: now also JP35.1, JP39.4, U1.B6; no longer JP13.1
- net COM2_TX/50HZ: now also JP20.4, JP36.1, JP40.1, U1.B5; no longer JP14.1
- net GND: now also C13.2, C14.2, IC5.GND, J1.GND, J1.SHIELD1, J1.SHIELD2, J1.SHIELD3, J1.SHIELD4, J1.SHIELD5, J1.SHIELD6, JP10.1, JP12.2, JP16.4, JP17.1, JP20.2, JP37.3, JP40.2, JP41.1, JP9.1, U1.GND; no longer DC1.-VIN, DC1.-VOUT, JP12.1, JP15.1, JP19.1, SV1-2.S
- net MISO*: now also JP13.3, JP16.1, JP19.3, U1.A4; no longer IC1.(PCINT14/MISO)PB6, JP6.1, SV1-7.S
- net MOSI*: now also JP16.2, JP19.2, U1.A1; no longer IC1.(PCINT13/MOSI)PB5, JP6.4, SV1-11.S
- net N$1: now also JP36.2, JP37.2; no longer JP14.2, JP21.2
- net N$16: now also JP9.3; no longer JP12.3
- net N$17: now also JP35.2, JP37.4; no longer JP13.2, JP21.4
- net N$3: now also JP9.2; no longer JP12.2
- net N$35: no longer DC1.+VIN
- net SCK*: now also JP15.4, JP19.1, U1.A3; no longer IC1.(PCINT15/SCK)PB7, JP6.3, SV1-8.S
- net SCL: now also JP35.3; no longer JP13.3
- net SCL_IN: now also JP41.4; no longer JP19.4
- net SCS*: now also JP15.3, JP18.4, U1.A2; no longer IC1.(PCINT12/OC0B/!SS!)PB4, SV1-9.S
- net SDA_IN: now also JP41.3; no longer JP19.3
- net VCC: now also C13.1, IC5.VI, J1.VBUS, JP10.3, JP12.1, JP36.3, JP37.1, JP40.3, U1.VCCB; no longer JP14.3, SV1-1.S
- net VDD: now also C14.1, IC5.VO, JP16.3, JP17.2, JP41.2, U1.OE, U1.VCCA; no longer DC1.+VOUT, JP19.2, SV1-10.S
Other:
- note added: "JP30 JP31 SD"
- note added: "JP37 JP38 50Hz Air UI Dust"
- note added: "JP39 JP40 GPS"
- note added: "JP41 Light Klima"
- note removed: "JP19 Light Klima"
- note removed: "JP21 JP22 50Hz Air UI Dust"
- moved on the sheet: C12, JP11, JP12, JP13, JP14, JP19, JP21, JP5
